Commit message: added exact position of the laserscanner on the real robot

File: stummel_urdf/defs/stummel_body.xacro (robot description, xacro)
@@ -366,5 +366,5 @@
         <xacro:include filename="$(find velodyne_description)/urdf/VLP-16.urdf.xacro"/>
         <VLP-16 parent="top_plate" name="velodyne" topic="/velodyne_points" hz="40" samples="440" gpu="${gpu}">
-            <origin xyz="0 0 0.4" rpy="0 0 0"/>
+            <origin xyz="0.125 0 0.34" rpy="0 0 3.14"/>
         </VLP-16>
     </xacro:macro>
