Commit message: experimental changes

File: stummel_urdf/defs/stummel.gazebo.xacro (robot description, xacro)
@@ -10,4 +10,6 @@
     <xacro:p3at_back suffix="left" reflect="1"/>
     <xacro:p3at_back suffix="right" reflect="-1"/>
+    <xacro:p3at_gazebo_ext/>
     <xacro:velodyne/>
+    <xacro:stummel_ground_truth_pose/>
 </robot>

File: stummel_urdf/defs/stummel_body.xacro (robot description, xacro)
@@ -4,363 +4,6 @@
 >
     <xacro:arg name="gpu" default="false"/>
-    <xacro:property name="gpu" value="$(arg gpu)"/>
-    <!-- Chassis -->
-    <link name="base_link">
-        <inertial>
-            <mass value="10.0"/>
-            <origin xyz="0 0 0.177"/>
-            <inertia ixx="0.3338" ixy="0.0" ixz="0.0"
-                     iyy="0.4783" iyz="0.0"
-                     izz="0.3338"/>
-        </inertial>
-        <visual name="base_visual">
-            <origin xyz="0 0 0.177" rpy="0 0 0"/>
-            <geometry name="pioneer_geom">
-                <mesh filename="package://p2os_urdf/meshes/p3at_meshes/chassis.stl"/>
-            </geometry>
-            <material name="ChassisRed">
-                <color rgba="0.851 0.0 0.0 1.0"/>
-            </material>
-        </visual>
-        <collision>
-            <origin xyz="0 0 0.177" rpy="0 0 0"/>
-            <geometry>
-                <mesh filename="package://p2os_urdf/meshes/p3at_meshes/chassis.stl"/>
-            </geometry>
-        </collision>
-    </link>
-    <gazebo reference="base_link">
-        <material value="Gazebo/Red"/>
-    </gazebo>
-    <!-- Top -->
-    <link name="top_plate">
-        <inertial>
-            <mass value="0.1"/>
-            <origin xyz="-0.025 0 -0.223"/>
-            <inertia ixx="1.0" ixy="0.0" ixz="0.0"
-                     iyy="1.0" iyz="0.0"
-                     izz="1.0"/>
-        </inertial>
-        <visual name="base_visual">
-            <origin xyz="0 0 0" rpy="0 0 0"/>
-            <geometry name="pioneer_geom">
-                <mesh filename="package://p2os_urdf/meshes/p3at_meshes/top.stl"/>
-            </geometry>
-            <material name="TopBlack">
-                <color rgba="0.038 0.038 0.038 1.0"/>
-            </material>
-        </visual>
-        <collision>
-            <origin xyz="0 0 0" rpy="0 0 0"/>
-            <geometry>
-                <box size="0 0 0"/>
-            </geometry>
-        </collision>
-    </link>
-    <gazebo reference="top_plate">
-        <material value="Gazebo/Black"/>
-    </gazebo>
-    <joint name="base_top_joint" type="fixed">
-        <origin xyz="0.003 0 0.274" rpy="0 0 0"/>
-        <parent link="base_link"/>
-        <child link="top_plate"/>
-    </joint>
-    <!-- Front + Back Sonar -->
-    <link name="front_sonar">
-        <inertial>
-            <mass value="0.1"/>
-            <origin xyz="0 0 0"/>
-            <inertia ixx="1.0" ixy="0.0" ixz="0.0"
-                     iyy="1.0" iyz="0.0" izz="1.0"/>
-        </inertial>
-        <visual name="base_visual">
-            <origin xyz="0 0 0" rpy="0 0 0"/>
-            <geometry name="pioneer_geom">
-                <mesh filename="package://p2os_urdf/meshes/p3at_meshes/front_sonar.stl"/>
-            </geometry>
-            <material name="SonarYellow">
-                <color rgba="0.715 0.583 0.210 1.0"/>
-            </material>
-        </visual>
-        <collision>
-            <origin xyz="0 0 0" rpy="0 0 0"/>
-            <geometry>
-                <box size="0 0 0"/>
-            </geometry>
-        </collision>
-    </link>
-    <gazebo reference="front_sonar">
-        <material value="Gazebo/Yellow"/>
-    </gazebo>
-    <joint name="base_front_joint" type="fixed">
-        <origin xyz="0.193 0 0.25" rpy="0 0 0"/>
-        <parent link="base_link"/>
-        <child link="front_sonar"/>
-    </joint>
-    <link name="back_sonar">
-        <inertial>
-            <mass value="0.1"/>
-            <origin xyz="0 0 0"/>
-            <inertia ixx="1.0" ixy="0.0" ixz="0.0"
-                     iyy="1.0" iyz="0.0" izz="1.0"/>
-        </inertial>
-        <visual name="base_visual">
-            <origin xyz="0 0 0" rpy="0 0 0"/>
-            <geometry name="pioneer_geom">
-                <mesh filename="package://p2os_urdf/meshes/p3at_meshes/back_sonar.stl"/>
-            </geometry>
-            <material name="SonarYellow">
-                <color rgba="0.715 0.583 0.210 1.0"/>
-            </material>
-        </visual>
-        <collision>
-            <origin xyz="0 0 0" rpy="0 0 0"/>
-            <geometry>
-                <box size="0 0 0"/>
-            </geometry>
-        </collision>
-    </link>
-    <gazebo reference="back_sonar">
-        <material value="Gazebo/Yellow"/>
-    </gazebo>
-    <joint name="base_back_joint" type="fixed">
-        <origin xyz="-0.187 0 0.247" rpy="0 0 0"/>
-        <parent link="base_link"/>
-        <child link="back_sonar"/>
-    </joint>
-    <!-- Front Axles + Wheels + Hubcaps -->
-    <xacro:macro name="p3at_front" params="suffix reflect">
-        <link name="p3at_front_${suffix}_axle">
-            <inertial>
-                <mass value="0.1"/>
-                <origin xyz="0 0 0"/>
-                <inertia ixx="1.0" ixy="0.0" ixz="0.0"
-                         iyy="1.0" iyz="0.0" izz="1.0"/>
-            </inertial>
-            <visual name="base_visual">
-                <origin xyz="0 0 0" rpy="0 0 0"/>
-                <geometry name="pioneer_geom">
-                    <mesh filename="package://p2os_urdf/meshes/p3at_meshes/axle.stl"/>
-                </geometry>
-                <material name="AxleGrey">
-                    <color rgba="0.5 0.5 0.5 1"/>
-                </material>
-            </visual>
-            <collision>
-                <origin xyz="0 0 0" rpy="0 0 0"/>
-                <geometry>
-                    <box size="0 0 0"/>
-                </geometry>
-            </collision>
-        </link>
-        <gazebo reference="p3at_front_${suffix}_axle">
-            <material value="Gazebo/Grey"/>
-        </gazebo>
-        <joint name="base_front_${suffix}_axle_joint" type="fixed">
-            <origin xyz="0.135 ${reflect*0.156} 0.111" rpy="0 0 0"/>
-            <parent link="base_link"/>
-            <child link="p3at_front_${suffix}_axle"/>
-        </joint>
-        <link name="p3at_front_${suffix}_hub">
-            <inertial>
-                <mass value="0.1"/>
-                <origin xyz="0 0 0"/>
-                <inertia ixx="1.0" ixy="0.0" ixz="0.0"
-                         iyy="1.0" iyz="0.0" izz="1.0"/>
-            </inertial>
-            <visual name="base_visual">
-                <origin xyz="0 0 0" rpy="0 0 0"/>
-                <geometry name="pioneer_geom">
-                    <mesh filename="package://p2os_urdf/meshes/p3at_meshes/${suffix}_hubcap.stl"/>
-                </geometry>
-                <material name="HubcapYellow">
-                    <color rgba="1.0 0.811 0.151 1.0"/>
-                </material>
-            </visual>
-            <collision>
-                <origin xyz="0 0 0" rpy="0 0 0"/>
-                <geometry>
-                    <box size="0 0 0"/>
-                </geometry>
-            </collision>
-        </link>
-        <gazebo reference="p3at_front_${suffix}_hub">
-            <material value="Gazebo/Yellow"/>
-        </gazebo>
-        <joint name="base_front_${suffix}_hub_joint" type="fixed">
-            <origin xyz="0 ${reflect*0.041} 0" rpy="0 0 0"/>
-            <parent link="p3at_front_${suffix}_axle"/>
-            <child link="p3at_front_${suffix}_hub"/>
-        </joint>
-        <link name="p3at_front_${suffix}_wheel">
-            <inertial>
-                <mass value="0.5"/>
-                <origin xyz="0 0 0"/>
-                <inertia ixx="0.012411765597" ixy="0" ixz="0"
-                         iyy="0.015218160428" iyz="0" izz="0.011763977943"/>
-            </inertial>
-            <visual name="base_visual">
-                <origin xyz="0 0 0" rpy="0 0 0"/>
-                <geometry name="pioneer_geom">
-                    <mesh filename="package://p2os_urdf/meshes/p3at_meshes/wheel.stl"/>
-                </geometry>
-                <material name="WheelBlack">
-                    <color rgba="0.117 0.117 0.117 1"/>
-                </material>
-            </visual>
-            <collision>
-                <origin xyz="0 0 0" rpy="${-3.1415927/2} 0 0"/>
-                <geometry>
-                    <!--mesh filename="package://p2os_urdf/meshes/p3at_meshes/wheel.stl"/-->
-                    <cylinder radius="0.111" length="0.075"/>
-                </geometry>
-            </collision>
-        </link>
-        <gazebo reference="p3at_front_${suffix}_wheel">
-            <material value="Gazebo/Black"/>
-        </gazebo>
-        <joint name="p3at_front_${suffix}_wheel_joint" type="continuous">
-            <axis xyz="0 1 0"/>
-            <anchor xyz="0 0 0"/>
-            <limit effort="100" velocity="100"/>
-            <joint_properties damping="0.7"/>
-            <origin xyz="0 0 0" rpy="0 0 0"/>
-            <parent link="p3at_front_${suffix}_hub"/>
-            <child link="p3at_front_${suffix}_wheel"/>
-        </joint>
-    </xacro:macro>
-    <!-- Back Axles + Wheels + Hubcaps -->
-    <xacro:macro name="p3at_back" params="suffix reflect">
-        <link name="p3at_back_${suffix}_axle">
-            <inertial>
-                <mass value="0.1"/>
-                <origin xyz="0 0 0"/>
-                <inertia ixx="1.0" ixy="0.0" ixz="0.0"
-                         iyy="1.0" iyz="0.0" izz="1.0"/>
-            </inertial>
-            <visual name="base_visual">
-                <origin xyz="0 0 0" rpy="0 0 0"/>
-                <geometry name="pioneer_geom">
-                    <mesh filename="package://p2os_urdf/meshes/p3at_meshes/axle.stl"/>
-                </geometry>
-                <material name="AxleGrey">
-                    <color rgba="0.5 0.5 0.5 1"/>
-                </material>
-            </visual>
-            <collision>
-                <origin xyz="0 0 0" rpy="0 0 0"/>
-                <geometry>
-                    <mesh filename="package://p2os_urdf/meshes/p3at_meshes/axle.stl"/>
-                </geometry>
-            </collision>
-        </link>
-        <gazebo reference="p3at_back_${suffix}_axle">
-            <material value="Gazebo/Grey"/>
-        </gazebo>
-        <joint name="bp3at_back_${suffix}_axle_joint" type="fixed">
-            <origin xyz="-0.134 ${reflect*0.156} 0.111" rpy="0 0 0"/>
-            <parent link="base_link"/>
-            <child link="p3at_back_${suffix}_axle"/>
-        </joint>
-        <link name="p3at_back_${suffix}_hub">
-            <inertial>
-                <mass value="0.1"/>
-                <origin xyz="0 0 0"/>
-                <inertia ixx="1.0" ixy="0.0" ixz="0.0"
-                         iyy="1.0" iyz="0.0" izz="1.0"/>
-            </inertial>
-            <visual name="base_visual">
-                <origin xyz="0 0 0" rpy="0 0 0"/>
-                <geometry name="pioneer_geom">
-                    <mesh filename="package://p2os_urdf/meshes/p3at_meshes/${suffix}_hubcap.stl"/>
-                </geometry>
-                <material name="HubcapYellow"/>
-            </visual>
-            <collision>
-                <origin xyz="0 0 0" rpy="0 0 0"/>
-                <geometry>
-                    <mesh filename="package://p2os_urdf/meshes/p3at_meshes/${suffix}_hubcap.stl"/>
-                </geometry>
-            </collision>
-        </link>
-        <gazebo reference="p3at_back_${suffix}_hub">
-            <material value="Gazebo/Yellow"/>
-        </gazebo>
-        <joint name="p3at_back_${suffix}_hub_joint" type="fixed">
-            <origin xyz="-0 ${reflect*0.041} 0" rpy="0 0 0"/>
-            <parent link="p3at_back_${suffix}_axle"/>
-            <child link="p3at_back_${suffix}_hub"/>
-        </joint>
-        <link name="p3at_back_${suffix}_wheel">
-            <inertial>
-                <mass value="0.5"/>
-                <origin xyz="0 0 0"/>
-                <inertia ixx="0.012411765597" ixy="0" ixz="0"
-                         iyy="0.015218160428" iyz="0" izz="0.011763977943"/>
-            </inertial>
-            <visual name="base_visual">
-                <origin xyz="0 0 0" rpy="0 0 0"/>
-                <geometry name="pioneer_geom">
-                    <mesh filename="package://p2os_urdf/meshes/p3at_meshes/wheel.stl"/>
-                </geometry>
-                <material name="WheelBlack"/>
-            </visual>
-            <collision>
-                <origin xyz="0 0 0" rpy="${-3.1415927/2} 0 0"/>
-                <geometry>
-                    <!--mesh filename="package://p2os_urdf/meshes/p3at_meshes/wheel.stl"/-->
-                    <cylinder radius="0.111" length="0.075"/>
-                </geometry>
-            </collision>
-        </link>
-        <gazebo reference="p3at_back_${suffix}_wheel">
-            <material value="Gazebo/Black"/>
-        </gazebo>
-        <joint name="p3at_back_${suffix}_wheel_joint" type="continuous">
-            <axis xyz="0 1 0"/>
-            <anchor xyz="0 0 0"/>
-            <limit effort="100" velocity="100"/>
-            <joint_properties damping="0.7"/>
-            <origin xyz="0 0 0" rpy="0 0 0"/>
-            <parent link="p3at_back_${suffix}_hub"/>
-            <child link="p3at_back_${suffix}_wheel"/>
-        </joint>
-        <gazebo reference="p3at_back_${suffix}_wheel">
-            <kp>1000000.0</kp> <!-- kp and kd for rubber -->
-            <kd>100.0</kd>
-            <mu1>10.0</mu1>
-            <mu2>1.0</mu2>
-            <fdir1>0 1 0</fdir1> <!-- is this correct? -->
-            <maxVel>1.0</maxVel>
-            <minDepth>0.00</minDepth>
-        </gazebo>
-        <gazebo reference="p3at_front_${suffix}_wheel">
-            <kp>1000000.0</kp> <!-- kp and kd for rubber -->
-            <kd>100.0</kd>
-            <mu1>10.0</mu1>
-            <mu2>1.0</mu2>
-            <fdir1>0 1 0</fdir1> <!-- is this correct? -->
-            <maxVel>1.0</maxVel>
-            <minDepth>0.00</minDepth>
-        </gazebo>
-    </xacro:macro>
-    <xacro:macro name="p3at_gazebo_ext">
-        <gazebo>
-            <plugin name="skid_steer_drive_controller" filename="libgazebo_ros_skid_steer_drive.so">
-                <updateRate>100.0</updateRate>
-                <robotNamespace>/</robotNamespace>
-                <leftFrontJoint>p3at_front_left_wheel_joint</leftFrontJoint>
-                <rightFrontJoint>p3at_front_right_wheel_joint</rightFrontJoint>
-                <leftRearJoint>p3at_back_left_wheel_joint</leftRearJoint>
-                <rightRearJoint>p3at_back_right_wheel_joint</rightRearJoint>
-                <wheelSeparation>0.4</wheelSeparation>
-                <wheelDiameter>0.215</wheelDiameter>
-                <robotBaseFrame>base_link</robotBaseFrame>
-                <torque>20</torque>
-                <broadcastTF>true</broadcastTF>
-                <topicName>cmd_vel</topicName>
-            </plugin>
-        </gazebo>
-    </xacro:macro>
+<xacro:property name="gpu" value="$(arg gpu)"/>
+    <xacro:include filename="$(find p2os_urdf)/defs/pioneer3at_body.xacro" />
     <xacro:macro name="velodyne">
         <xacro:include filename="$(find velodyne_description)/urdf/VLP-16.urdf.xacro"/>

Commit message: moved simulated velodyne out of real body

File: stummel_urdf/defs/stummel.gazebo.xacro (robot description, xacro)
@@ -6,4 +6,24 @@
        name="stummel_sim">
     <xacro:include filename="$(find cnc-stummeldriver)/stummel_urdf/defs/stummel_body.xacro"/>
+ <!-- Makes Gazebo publishing a ground truth position. -->
+  <xacro:macro name="stummel_ground_truth_pose">
+    <gazebo>
+      <plugin name="p3d_controller" filename="libgazebo_ros_p3d.so">
+       <alwaysOn>true</alwaysOn>
+       <updateRate>100.0</updateRate>
+       <bodyName>base_link</bodyName>
+       <topicName>ground_truth_pose</topicName>
+       <frameName>/map</frameName>
+       <xyzOffsets>1 1 0</xyzOffsets> <!-- option to initialize odometry for fake localization-->
+       <rpyOffsets>0 0 0</rpyOffsets>
+      </plugin>
+    </gazebo>
+  </xacro:macro>
+    <xacro:macro name="velodyne">
+        <xacro:include filename="$(find velodyne_description)/urdf/VLP-16.urdf.xacro"/>
+        <VLP-16 parent="top_plate" name="velodyne" topic="/velodyne_points" hz="40" samples="440" gpu="${gpu}">
+            <origin xyz="0.125 0 0.34" rpy="0 0 3.14"/>
+        </VLP-16>
+    </xacro:macro>
     <xacro:p3at_front suffix="left" reflect="1"/>
     <xacro:p3at_front suffix="right" reflect="-1"/>

File: stummel_urdf/defs/stummel_body.xacro (robot description, xacro)
@@ -6,23 +6,3 @@
 <xacro:property name="gpu" value="$(arg gpu)"/>
     <xacro:include filename="$(find p2os_urdf)/defs/pioneer3at_body.xacro" />
-    <xacro:macro name="velodyne">
-        <xacro:include filename="$(find velodyne_description)/urdf/VLP-16.urdf.xacro"/>
-        <VLP-16 parent="top_plate" name="velodyne" topic="/velodyne_points" hz="40" samples="440" gpu="${gpu}">
-            <origin xyz="0 0 0.4" rpy="0 0 0"/>
-        </VLP-16>
-    </xacro:macro>
- <!-- Makes Gazebo publishing a ground truth position. -->
-  <xacro:macro name="stummel_ground_truth_pose">
-    <gazebo>
-      <plugin name="p3d_controller" filename="libgazebo_ros_p3d.so">
-       <alwaysOn>true</alwaysOn>
-       <updateRate>100.0</updateRate>
-       <bodyName>base_link</bodyName>
-       <topicName>ground_truth_pose</topicName>
-       <frameName>/map</frameName>
-       <xyzOffsets>1 1 0</xyzOffsets> <!-- option to initialize odometry for fake localization-->
-       <rpyOffsets>0 0 0</rpyOffsets>
-      </plugin>
-    </gazebo>
-  </xacro:macro>
 </robot>
